File: _autosave-blheli_esc.kicad_pcb (KiCad board)
At the start: 2 copper layers, 45 parts, among them J1 Conn_01x03_Male, Q1 BC847, Q2 BC847, Q3 BC847, U1 AP1509, U2 EFM8BB21F16G

Commit message: schematic mostly done, working on layout
Parts:
- moved TP1 68.0 mm to (152.5, 70.5)
- moved TP5 39.9 mm to (152.5, 68.2)
- moved TP3 37.7 mm to (155.6, 76.6)
- moved TP2 32.4 mm to (155.6, 74.5)
- moved D1 22.3 mm to (155.5, 78.8), turned to 180 degrees
Routing:
- net C2D: track 0.00 -> 5.28 mm
- net Net-(J1-Pad2): track 0.00 -> 3.88 mm
- net Net-(D1-Pad1): track 0.00 -> 2.15 mm
- net C2CK: track 2.27 -> 4.01 mm
- net RC_IN: track 15.6 -> 17.0 mm
Changed lines of the file:
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@@
     (thickness 1.6)
     (drawings 0)
-    (tracks 99)
+    (tracks 114)
     (zones 0)
     (modules 45)
@@
   )
   (module Diode_SMD:D_SOD-123F (layer F.Cu)
-    (at 139.5065 63.246)
+    (at 155.451 78.8035 180)
     (descr D_SOD-123F)
     (tags D_SOD-123F)
     (attr smd)
-    (fp_text reference D1 (at -0.127 -1.905) (layer F.SilkS)
-      (effects (font (size 1 1) (thickness 0.15)))
-    )
-    (fp_text value MBR120V (at 0 2.1) (layer F.Fab)
-      (effects (font (size 1 1) (thickness 0.15)))
-    )
-    (fp_text user %R (at -0.127 -1.905) (layer F.Fab)
+    (fp_text reference D1 (at -0.127 -1.905 180) (layer F.SilkS)
+      (effects (font (size 1 1) (thickness 0.15)))
+    )
+    (fp_text value MBR120V (at 0 2.1 180) (layer F.Fab)
+      (effects (font (size 1 1) (thickness 0.15)))
+    )
+    (fp_text user %R (at -0.127 -1.905 180) (layer F.Fab)
       (effects (font (size 1 1) (thickness 0.15)))
     )
@@
     (fp_line (start -2.2 1) (end 1.65 1) (layer F.SilkS) (width 0.12))
     (fp_line (start -2.2 -1) (end 1.65 -1) (layer F.SilkS) (width 0.12))
-    (pad 1 smd rect (at -1.4 0) (size 1.1 1.1) (layers F.Cu F.Paste F.Mask)
+    (pad 1 smd rect (at -1.4 0 180) (size 1.1 1.1) (layers F.Cu F.Paste F.Mask)
       (net 4 "Net-(D1-Pad1)"))
-    (pad 2 smd rect (at 1.4 0) (size 1.1 1.1) (layers F.Cu F.Paste F.Mask)
+    (pad 2 smd rect (at 1.4 0 180) (size 1.1 1.1) (layers F.Cu F.Paste F.Mask)
       (net 1 GND))
     (model ${KISYS3DMOD}/Diode_SMD.3dshapes/D_SOD-123F.wrl
@@
   )
   (module TestPoint:TestPoint_THTPad_D1.0mm_Drill0.5mm (layer F.Cu)
-    (at 107.95 121.92)
+    (at 152.4635 70.5485)
     (descr "THT pad as test Point, diameter 1.0mm, hole diameter 0.5mm")
     (tags "test point THT pad")
@@
   )
   (module TestPoint:TestPoint_THTPad_D1.0mm_Drill0.5mm (layer F.Cu)
-    (at 151.765 106.68)
+    (at 155.575 74.4855)
     (descr "THT pad as test Point, diameter 1.0mm, hole diameter 0.5mm")
     (tags "test point THT pad")
     (attr virtual)
-    (fp_text reference TP2 (at 0 -1.448) (layer F.SilkS)
+    (fp_text reference TP2 (at -2.159 0.1905) (layer F.SilkS)
       (effects (font (size 1 1) (thickness 0.15)))
     )
@@
   )
   (module TestPoint:TestPoint_THTPad_D1.0mm_Drill0.5mm (layer F.Cu)
-    (at 154.305 114.3)
+    (at 155.575 76.581)
     (descr "THT pad as test Point, diameter 1.0mm, hole diameter 0.5mm")
     (tags "test point THT pad")
     (attr virtual)
-    (fp_text reference TP3 (at 0 -1.448) (layer F.SilkS)
+    (fp_text reference TP3 (at 0.0635 1.7145) (layer F.SilkS)
       (effects (font (size 1 1) (thickness 0.15)))
     )
@@
   )
   (module TestPoint:TestPoint_THTPad_D1.0mm_Drill0.5mm (layer F.Cu)
-    (at 144.78 107.315)
+    (at 152.4635 68.199)
     (descr "THT pad as test Point, diameter 1.0mm, hole diameter 0.5mm")
     (tags "test point THT pad")
@@
   (segment (start 154.97799 71.85651) (end 156.15069 71.85651) (width 0.25) (layer F.Cu) (net 3))
   (segment (start 154.0635 72.771) (end 154.97799 71.85651) (width 0.25) (layer F.Cu) (net 3))
+  (segment (start 157.359 79.3115) (end 156.851 78.8035) (width 0.25) (layer F.Cu) (net 4))
+  (segment (start 158.7925 79.3115) (end 157.359 79.3115) (width 0.25) (layer F.Cu) (net 4))
   (segment (start 176.553 68.438) (end 176.403 68.588) (width 0.25) (layer F.Cu) (net 6))
   (segment (start 177.2655 68.438) (end 176.553 68.438) (width 0.25) (layer F.Cu) (net 6))
@@
   (segment (start 171.196 80.264) (end 171.653 80.264) (width 0.25) (layer F.Cu) (net 12))
   (segment (start 149.982 68.326) (end 148.717 68.326) (width 0.25) (layer F.Cu) (net 14))
-  (segment (start 159.86628 66.88548) (end 151.42252 66.88548) (width 0.25) (layer F.Cu) (net 14))
   (segment (start 161.8783 68.8975) (end 159.86628 66.88548) (width 0.25) (layer F.Cu) (net 14))
   (segment (start 151.42252 66.88548) (end 149.982 68.326) (width 0.25) (layer F.Cu) (net 14))
   (segment (start 162.9283 68.8975) (end 161.8783 68.8975) (width 0.25) (layer F.Cu) (net 14))
+  (segment (start 152.4635 67.491894) (end 152.4635 66.88548) (width 0.25) (layer F.Cu) (net 14))
+  (segment (start 152.4635 68.199) (end 152.4635 67.491894) (width 0.25) (layer F.Cu) (net 14))
+  (segment (start 159.86628 66.88548) (end 152.4635 66.88548) (width 0.25) (layer F.Cu) (net 14))
+  (segment (start 152.4635 66.88548) (end 151.42252 66.88548) (width 0.25) (layer F.Cu) (net 14))
+  (segment (start 152.146 70.866) (end 152.4635 70.5485) (width 0.25) (layer F.Cu) (net 15))
+  (segment (start 148.717 70.866) (end 152.146 70.866) (width 0.25) (layer F.Cu) (net 15))
   (segment (start 167.691 68.072) (end 166.116 69.647) (width 0.25) (layer F.Cu) (net 16))
   (segment (start 166.116 69.647) (end 166.116 70.104) (width 0.25) (layer F.Cu) (net 16))
@@
   (segment (start 156.100112 72.309388) (end 156.494699 72.309388) (width 0.25) (layer F.Cu) (net 19))
   (segment (start 155.6385 72.771) (end 156.100112 72.309388) (width 0.25) (layer F.Cu) (net 19))
+  (segment (start 155.575 72.8345) (end 155.6385 72.771) (width 0.25) (layer F.Cu) (net 19))
+  (segment (start 155.575 74.4855) (end 155.575 72.8345) (width 0.25) (layer F.Cu) (net 19))
   (segment (start 154.0635 71.0565) (end 154.0635 69.596) (width 0.25) (layer F.Cu) (net 20))
   (segment (start 154.0635 69.596) (end 154.0635 68.1355) (width 0.25) (layer F.Cu) (net 20))
@@
   (segment (start 156.4005 68.8975) (end 157.6197 68.8975) (width 0.25) (layer F.Cu) (net 23))
   (segment (start 155.6385 68.1355) (end 156.4005 68.8975) (width 0.25) (layer F.Cu) (net 23))
+  (segment (start 156.559699 72.812499) (end 157.514701 72.812499) (width 0.25) (layer F.Cu) (net 27))
+  (segment (start 156.494699 72.877499) (end 156.559699 72.812499) (width 0.25) (layer F.Cu) (net 27))
+  (segment (start 156.494699 74.786803) (end 156.494699 72.877499) (width 0.25) (layer F.Cu) (net 27))
+  (segment (start 155.575 75.706502) (end 156.494699 74.786803) (width 0.25) (layer F.Cu) (net 27))
+  (segment (start 157.514701 72.812499) (end 157.6197 72.7075) (width 0.25) (layer F.Cu) (net 27))
+  (segment (start 155.575 76.581) (end 155.575 75.706502) (width 0.25) (layer F.Cu) (net 27))
   (segment (start 163.703 68.2625) (end 164.719 67.2465) (width 0.25) (layer F.Cu) (net 28))
   (segment (start 162.9283 68.2625) (end 163.703 68.2625) (width 0.25) (layer F.Cu) (net 28))
