File: _saved_blheli_esc.sch (KiCad schematic (older format))
At the start: 42 parts, among them J1 Conn_01x03_Male, Q1 BC847, Q2 BC847, Q3 BC847, U1 AP1509, U2 EFM8BB21F16G

Commit message: schematic mostly done, working on layout
Parts:
- added TP6: PHASE_A, TestPoint:TestPoint_Pad_1.5x1.5mm, symbol Connector:TestPoint
- added TP7: PHASE_B, TestPoint:TestPoint_Pad_1.5x1.5mm, symbol Connector:TestPoint
- added TP8: PHASE_C, TestPoint:TestPoint_Pad_1.5x1.5mm, symbol Connector:TestPoint
Connections:
- net PHASE_A: now also TP6.1
- net PHASE_B: now also TP7.1
- net PHASE_C: now also TP8.1
Other:
- moved on the sheet: J1, TP1, TP2, TP3, TP4, TP5
Changed lines of the file:
@@
 L Connector:TestPoint TP2
 U 1 1 5C2EF43A
-P 3050 4200
-F 0 "TP2" V 3004 4387 50  0000 L CNN
-F 1 "C2CK" V 3095 4387 50  0000 L CNN
-F 2 "TestPoint:TestPoint_THTPad_D1.0mm_Drill0.5mm" H 3250 4200 50  0001 C CNN
-F 3 "~" H 3250 4200 50  0001 C CNN
-	1    3050 4200
-	0    1    1    0
-$EndComp
-Text GLabel 2850 4200 0    50   Input ~ 0
+P 3100 3550
+F 0 "TP2" V 3054 3737 50  0000 L CNN
+F 1 "C2CK" V 3145 3737 50  0000 L CNN
+F 2 "TestPoint:TestPoint_THTPad_D1.0mm_Drill0.5mm" H 3300 3550 50  0001 C CNN
+F 3 "~" H 3300 3550 50  0001 C CNN
+	1    3100 3550
+	0    1    1    0
+$EndComp
+Text GLabel 2900 3550 0    50   Input ~ 0
 C2CK
 Wire Wire Line
-	2850 4200 3050 4200
+	2900 3550 3100 3550
 $Comp
 L Connector:TestPoint TP3
 U 1 1 5C2F3D95
-P 3050 4400
-F 0 "TP3" V 3004 4587 50  0000 L CNN
-F 1 "C2D" V 3095 4587 50  0000 L CNN
-F 2 "TestPoint:TestPoint_THTPad_D1.0mm_Drill0.5mm" H 3250 4400 50  0001 C CNN
-F 3 "~" H 3250 4400 50  0001 C CNN
-	1    3050 4400
-	0    1    1    0
-$EndComp
-Text GLabel 2850 4400 0    50   Input ~ 0
+P 3100 3750
+F 0 "TP3" V 3054 3937 50  0000 L CNN
+F 1 "C2D" V 3145 3937 50  0000 L CNN
+F 2 "TestPoint:TestPoint_THTPad_D1.0mm_Drill0.5mm" H 3300 3750 50  0001 C CNN
+F 3 "~" H 3300 3750 50  0001 C CNN
+	1    3100 3750
+	0    1    1    0
+$EndComp
+Text GLabel 2900 3750 0    50   Input ~ 0
 C2D
 Wire Wire Line
-	2850 4400 3050 4400
-Text GLabel 2850 4600 0    50   Input ~ 0
+	2900 3750 3100 3750
+Text GLabel 2900 3950 0    50   Input ~ 0
 TX2
 $Comp
 L Connector:TestPoint TP4
 U 1 1 5C2F885D
-P 3050 4600
-F 0 "TP4" V 3004 4788 50  0000 L CNN
-F 1 "TX2" V 3095 4788 50  0000 L CNN
-F 2 "TestPoint:TestPoint_THTPad_D1.0mm_Drill0.5mm" H 3250 4600 50  0001 C CNN
-F 3 "~" H 3250 4600 50  0001 C CNN
-	1    3050 4600
-	0    1    1    0
-$EndComp
-Wire Wire Line
-	2850 4600 3050 4600
-Text GLabel 2850 4800 0    50   Output ~ 0
+P 3100 3950
+F 0 "TP4" V 3054 4138 50  0000 L CNN
+F 1 "TX2" V 3145 4138 50  0000 L CNN
+F 2 "TestPoint:TestPoint_THTPad_D1.0mm_Drill0.5mm" H 3300 3950 50  0001 C CNN
+F 3 "~" H 3300 3950 50  0001 C CNN
+	1    3100 3950
+	0    1    1    0
+$EndComp
+Wire Wire Line
+	2900 3950 3100 3950
+Text GLabel 2900 4150 0    50   Output ~ 0
 RC_IN
 $Comp
 L Connector:TestPoint TP5
 U 1 1 5C2FD85C
-P 3050 4800
-F 0 "TP5" V 3004 4987 50  0000 L CNN
-F 1 "RC_IN" V 3095 4987 50  0000 L CNN
-F 2 "TestPoint:TestPoint_THTPad_D1.0mm_Drill0.5mm" H 3250 4800 50  0001 C CNN
-F 3 "~" H 3250 4800 50  0001 C CNN
-	1    3050 4800
-	0    1    1    0
-$EndComp
-Wire Wire Line
-	2850 4800 3050 4800
+P 3100 4150
+F 0 "TP5" V 3054 4337 50  0000 L CNN
+F 1 "RC_IN" V 3145 4337 50  0000 L CNN
+F 2 "TestPoint:TestPoint_THTPad_D1.0mm_Drill0.5mm" H 3300 4150 50  0001 C CNN
+F 3 "~" H 3300 4150 50  0001 C CNN
+	1    3100 4150
+	0    1    1    0
+$EndComp
+Wire Wire Line
+	2900 4150 3100 4150
 $Comp
 L Connector:Conn_01x03_Male J1
 U 1 1 5C302F31
-P 1200 4400
-F 0 "J1" H 1306 4678 50  0000 C CNN
-F 1 "Conn_01x03_Male" H 1306 4587 50  0000 C CNN
-F 2 "Connector:FanPinHeader_1x03_P2.54mm_Vertical" H 1200 4400 50  0001 C CNN
-F 3 "~" H 1200 4400 50  0001 C CNN
-	1    1200 4400
+P 1100 3800
+F 0 "J1" H 1206 4078 50  0000 C CNN
+F 1 "Conn_01x03_Male" H 1206 3987 50  0000 C CNN
+F 2 "Connector:FanPinHeader_1x03_P2.54mm_Vertical" H 1100 3800 50  0001 C CNN
+F 3 "~" H 1100 3800 50  0001 C CNN
+	1    1100 3800
 	1    0    0    -1
 $EndComp
@@
 L power:GND #PWR0112
 U 1 1 5C30CB8C
-P 1500 4600
-F 0 "#PWR0112" H 1500 4350 50  0001 C CNN
-F 1 "GND" H 1505 4427 50  0000 C CNN
-F 2 "" H 1500 4600 50  0001 C CNN
-F 3 "" H 1500 4600 50  0001 C CNN
-	1    1500 4600
-	1    0    0    -1
-$EndComp
-Wire Wire Line
-	1400 4500 1500 4500
-Text GLabel 1600 4300 2    50   Output ~ 0
+P 1400 4000
+F 0 "#PWR0112" H 1400 3750 50  0001 C CNN
+F 1 "GND" H 1405 3827 50  0000 C CNN
+F 2 "" H 1400 4000 50  0001 C CNN
+F 3 "" H 1400 4000 50  0001 C CNN
+	1    1400 4000
+	1    0    0    -1
+$EndComp
+Wire Wire Line
+	1300 3900 1400 3900
+Text GLabel 1500 3700 2    50   Output ~ 0
 RC_IN
 Wire Wire Line
-	1400 4300 1600 4300
+	1300 3700 1500 3700
 $Comp
 L Connector:TestPoint TP1
 U 1 1 5C32EFFC
-P 1400 4400
-F 0 "TP1" V 1354 4587 50  0000 L CNN
-F 1 "SERVO_TP" V 1445 4587 50  0000 L CNN
-F 2 "TestPoint:TestPoint_THTPad_D1.0mm_Drill0.5mm" H 1600 4400 50  0001 C CNN
-F 3 "~" H 1600 4400 50  0001 C CNN
-	1    1400 4400
-	0    1    1    0
-$EndComp
-Wire Wire Line
-	1500 4600 1500 4500
+P 1300 3800
+F 0 "TP1" V 1254 3987 50  0000 L CNN
+F 1 "SERVO_TP" V 1345 3987 50  0000 L CNN
+F 2 "TestPoint:TestPoint_THTPad_D1.0mm_Drill0.5mm" H 1500 3800 50  0001 C CNN
+F 3 "~" H 1500 3800 50  0001 C CNN
+	1    1300 3800
+	0    1    1    0
+$EndComp
+Wire Wire Line
+	1400 4000 1400 3900
 $Comp
 L blheli_esc:PAD PAD1
@@
 	5700 1750 6300 1750
 Connection ~ 5700 1750
+Text GLabel 2900 4600 0    50   Input ~ 0
+PHASE_A
+Text GLabel 2900 4900 0    50   Input ~ 0
+PHASE_B
+Text GLabel 2900 5200 0    50   Input ~ 0
+PHASE_C
+$Comp
+L Connector:TestPoint TP6
+U 1 1 5C42D9CE
+P 3100 4600
+F 0 "TP6" V 3054 4788 50  0000 L CNN
+F 1 "PHASE_A" V 3145 4788 50  0000 L CNN
+F 2 "TestPoint:TestPoint_Pad_1.5x1.5mm" H 3300 4600 50  0001 C CNN
+F 3 "~" H 3300 4600 50  0001 C CNN
+	1    3100 4600
+	0    1    1    0
+$EndComp
+$Comp
+L Connector:TestPoint TP7
+U 1 1 5C42DAE7
+P 3100 4900
+F 0 "TP7" V 3054 5087 50  0000 L CNN
+F 1 "PHASE_B" V 3145 5087 50  0000 L CNN
+F 2 "TestPoint:TestPoint_Pad_1.5x1.5mm" H 3300 4900 50  0001 C CNN
+F 3 "~" H 3300 4900 50  0001 C CNN
+	1    3100 4900
+	0    1    1    0
+$EndComp
+$Comp
+L Connector:TestPoint TP8
+U 1 1 5C42DC72
+P 3100 5200
+F 0 "TP8" V 3054 5387 50  0000 L CNN
+F 1 "PHASE_C" V 3145 5387 50  0000 L CNN
+F 2 "TestPoint:TestPoint_Pad_1.5x1.5mm" H 3300 5200 50  0001 C CNN
+F 3 "~" H 3300 5200 50  0001 C CNN
+	1    3100 5200
+	0    1    1    0
+$EndComp
+Wire Wire Line
+	2900 4600 3100 4600
+Wire Wire Line
+	2900 4900 3100 4900
+Wire Wire Line
+	2900 5200 3100 5200
 $EndSCHEMATC
